Commit message: modify the dead file and rviz

File: src/mobile_robot_description/urdf/camera.xacro (robot description, xacro)
@@ -8,10 +8,10 @@
         <parent link="base_link"/>
         <child link="camera_link"/>
-        <origin xyz="0.305 0 0.08" rpy="0 0 0"/>
+        <origin xyz="0.05 0 0.04" rpy="0 0 0"/>
     </joint>
     <link name="camera_link">
         <visual>
             <geometry>
-                <box size="0.010 0.03 0.03"/>
+                <box size="0.005 0.015 0.015"/>
             </geometry>
             <material name="red"/>
@@ -21,5 +21,5 @@
         <parent link="camera_link"/>
         <child link="camera_link_optical"/>
-        <origin xyz="0 0 0" rpy="${-pi/2} 0 ${-pi/2}"/>
+        <origin xyz="0 0 0" rpy="-1.57 0 0"/>
     </joint>
     <link name="camera_link_optical"></link>
